File: audioserial.sch (KiCad schematic (older format))
At the start: 19 parts

Commit message: current
Parts:
- removed J?: USB, symbol USB
- removed L?: SRF2012, symbol SRF2012
- removed R?: 10K, symbol R
- removed U?: FT232RL, symbol FT232RL
- added P?: CONN_SERIAL, symbol CONN_01X05
- added U?: MAX232, symbol MAX232
Connections:
- net at U?.42 (PA9): now also P?.5 (P5)
- net at U?.43 (PA10): now also P?.4 (P4)
- net at U?.44 (PA11): now also P?.3 (P3)
- net at U?.45 (PA12): now also P?.2 (P2)
- net at U?.46 (PA13): now also P?.1 (P1)
Changed lines of the file:
@@
 $EndComp
-$Comp
-L R R?
-U 1 1 540ADCFF
-P 6950 3100
-F 0 "R?" V 7030 3100 40  0000 C CNN
-F 1 "10K" V 6957 3101 40  0000 C CNN
-F 2 "" V 6880 3100 30  0000 C CNN
-F 3 "" H 6950 3100 30  0000 C CNN
-	1    6950 3100
-	1    0    0    -1
-$EndComp
-Wire Wire Line
-	6250 3350 6950 3350
-$Comp
-L +3.3V #PWR?
-U 1 1 540ADD96
-P 6950 2700
-F 0 "#PWR?" H 6950 2660 30  0001 C CNN
-F 1 "+3.3V" H 6950 2810 30  0000 C CNN
-F 2 "" H 6950 2700 60  0000 C CNN
-F 3 "" H 6950 2700 60  0000 C CNN
-	1    6950 2700
-	1    0    0    -1
-$EndComp
-Wire Wire Line
-	6950 2700 6950 2850
 $Comp
 L CRYSTAL X?
@@
 Wire Wire Line
 	2350 5600 1850 5600
-$Comp
-L FT232RL U?
-U 1 1 540B0652
-P 9250 1600
-F 0 "U?" H 9250 2500 60  0000 C CNN
-F 1 "FT232RL" H 9650 600 60  0000 L CNN
-F 2 "" H 9250 1600 60  0000 C CNN
-F 3 "" H 9250 1600 60  0000 C CNN
-	1    9250 1600
-	1    0    0    -1
-$EndComp
-Wire Wire Line
-	8950 2800 9550 2800
-Connection ~ 9400 2800
-Connection ~ 9250 2800
-Connection ~ 9100 2800
-Wire Wire Line
-	8950 2800 8950 3000
-$Comp
-L GND #PWR?
-U 1 1 540B095A
-P 8950 3000
-F 0 "#PWR?" H 8950 3000 30  0001 C CNN
-F 1 "GND" H 8950 2930 30  0001 C CNN
-F 2 "" H 8950 3000 60  0000 C CNN
-F 3 "" H 8950 3000 60  0000 C CNN
-	1    8950 3000
-	1    0    0    -1
-$EndComp
-$Comp
-L USB J?
-U 1 1 540B0A3A
-P 6650 950
-F 0 "J?" H 6600 1350 60  0000 C CNN
-F 1 "USB" V 6400 1100 60  0000 C CNN
-F 2 "" H 6650 950 60  0000 C CNN
-F 3 "" H 6650 950 60  0000 C CNN
-	1    6650 950
-	1    0    0    -1
-$EndComp
-$Comp
-L SRF2012 L?
-U 1 1 540B1991
-P 7650 1150
-F 0 "L?" H 7650 1250 60  0000 C CNN
-F 1 "SRF2012" H 7650 850 60  0000 C CNN
-F 2 "" H 7650 1050 60  0000 C CNN
-F 3 "" H 7650 1050 60  0000 C CNN
-	1    7650 1150
-	1    0    0    -1
-$EndComp
-Wire Wire Line
-	8300 1200 8050 1200
-Wire Wire Line
-	8050 1200 8050 1150
-Wire Wire Line
-	8050 1150 7850 1150
-Wire Wire Line
-	7450 1150 7200 1150
-Wire Wire Line
-	7200 1150 7200 1300
-Wire Wire Line
-	7200 1300 7000 1300
-Wire Wire Line
-	7450 1350 7300 1350
-Wire Wire Line
-	7300 1350 7300 1200
-Wire Wire Line
-	7300 1200 7000 1200
-Wire Wire Line
-	7000 1200 7000 1150
-Wire Wire Line
-	7850 1350 8050 1350
-Wire Wire Line
-	8050 1350 8050 1300
-Wire Wire Line
-	8050 1300 8300 1300
+Wire Wire Line
+	6250 3350 7150 3350
+Wire Wire Line
+	6250 3250 7150 3250
+Wire Wire Line
+	6250 3150 7150 3150
+Wire Wire Line
+	6250 3050 7150 3050
+Wire Wire Line
+	6250 2950 7150 2950
+$Comp
+L CONN_01X05 P?
+U 1 1 540B29E0
+P 7350 3150
+F 0 "P?" H 7350 3450 50  0000 C CNN
+F 1 "CONN_SERIAL" V 7450 3150 50  0000 C CNN
+F 2 "" H 7350 3150 60  0000 C CNN
+F 3 "" H 7350 3150 60  0000 C CNN
+	1    7350 3150
+	1    0    0    -1
+$EndComp
+$Comp
+L MAX232 U?
+U 1 1 540B2E49
+P 9200 3650
+F 0 "U?" H 9200 4500 70  0000 C CNN
+F 1 "MAX232" H 9200 2800 70  0000 C CNN
+F 2 "" H 9200 3650 60  0000 C CNN
+F 3 "" H 9200 3650 60  0000 C CNN
+	1    9200 3650
+	1    0    0    -1
+$EndComp
 $EndSCHEMATC
